File: Hardware/CanSat2020ProbeS/CanSat2020Probe.sch (KiCad schematic (older format))
At the start: 33 parts, among them IC1 TESEO-LIV3F, J1 BME280, J2 MPU-9250, J3 Micro_SD_Card, J4 Conn_01x03_Male, J5 Conn_Coaxial, J6 Conn_Coaxial, J7 Conn_01x05_Male, J8 Conn_01x03_Male, U1 STM32F411RETx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

Commit message: addition of new components
Parts:
- C10: footprint Capacitor_SMD:CP_Elec_8x10 -> Capacitor_SMD:CP_Elec_5x5.3
- C8: footprint Capacitor_SMD:CP_Elec_8x10 -> Capacitor_THT:CP_Radial_D5.0mm_P2.00mm
Changed lines of the file:
@@
 F 0 "C8" H 3215 6746 50  0000 L CNN
 F 1 "47uF" H 3215 6655 50  0000 L CNN
-F 2 "Capacitor_SMD:CP_Elec_8x10" H 3138 6550 50  0001 C CNN
+F 2 "Capacitor_THT:CP_Radial_D5.0mm_P2.00mm" H 3138 6550 50  0001 C CNN
 F 3 "~" H 3100 6700 50  0001 C CNN
 	1    3100 6700
@@
 F 0 "C10" H 4565 6746 50  0000 L CNN
 F 1 "47uF" H 4565 6655 50  0000 L CNN
-F 2 "Capacitor_SMD:CP_Elec_8x10" H 4488 6550 50  0001 C CNN
+F 2 "Capacitor_SMD:CP_Elec_5x5.3" H 4488 6550 50  0001 C CNN
 F 3 "~" H 4450 6700 50  0001 C CNN
 	1    4450 6700
