File: Probe/Hardware/CanSat2020ProbeS/CanSat2020Probe.kicad_pcb (KiCad board)
At the start: 2 copper layers, 33 parts, among them IC1 TESEO-LIV3F, J1 BME280, J2 MPU-9250, J3 Micro_SD_Card, J4 Conn_01x03_Male, J5 Conn_Coaxial, J6 Conn_Coaxial, J7 Conn_01x05_Male, J8 Conn_01x03_Male, U1 STM32F411RETx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

Commit message: upadte
Parts:
- added C11: 4.7uF, Capacitor_SMD:C_0805_2012Metric, F.Cu at (153.3, 104.8)
- added SW1: SW_DIP_x01, Switch:Sw1, B.Cu at (126.2, 100.0)
- C6, D1, D2, D3, J3, R3, R4, R5: moved to B.Cu
- J1: footprint Connector_PinHeader_2.54mm:PinHeader_1x04_P2.54mm_Vertical -> Switch:BME280; moved to B.Cu
- J2: footprint Connector_PinHeader_2.54mm:PinHeader_1x10_P2.54mm_Vertical -> Switch:MPU-9250
- J5, J6: footprint Connector_Coaxial:U.FL_Molex_MCRF_73412-0110_Vertical -> Connector_Coaxial:U.FL_Hirose_U.FL-R-SMT-1_Vertical
- J8: value Conn_01x03_Male -> Conn_01x02_Male; footprint Connector_PinHeader_2.54mm:PinHeader_1x03_P2.54mm_Vertical -> Connector_PinHeader_2.54mm:PinHeader_1x02_P2.54mm_Vertical
- moved C7 123.2 mm to (167.1, 108.5), turned to 270 degrees
- moved D1 121.5 mm to (193.4, 104.2)
- moved J7 116.0 mm to (166.4, 90.4), turned to 180 degrees
- moved U2 115.7 mm to (155.0, 114.5), turned to 180 degrees
- moved J2 114.9 mm to (158.2, 78.8), turned to 270 degrees
- moved D3 114.2 mm to (193.4, 98.0)
- moved C6 107.7 mm to (144.4, 116.7), turned to 270 degrees
- moved C5 107.1 mm to (162.8, 79.8), turned to 90 degrees
- moved J3 102.0 mm to (154.7, 115.0), turned to 90 degrees
- moved D2 101.5 mm to (193.4, 101.0)
- moved R3 100.5 mm to (188.9, 104.2), turned to 180 degrees
- moved R4 95.9 mm to (188.9, 101.0), turned to 180 degrees
- moved C9 95.8 mm to (139.4, 106.6), turned to 270 degrees
- moved R5 95.0 mm to (188.9, 98.0), turned to 180 degrees
- moved J5 93.4 mm to (173.8, 106.1), turned to 270 degrees
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Connections:
- J4 pad 1: +BATT -> Net-(J4-Pad1)
- J8 pad 1: GND -> /DBGTX
- J8 pad 2: /DBGTX -> /DBGRX
Routing:
- net (no net): vias 0 -> 9
Other:
- board text added: "1 2 3"

Commit message: Impprovements
Routing:
- net Net-(C3-Pad2): track 0.00 -> 4.05 mm
- net Net-(C2-Pad1): track 0.00 -> 3.75 mm
Changed lines of the file:
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@@
     (thickness 1.6)
     (drawings 5)
-    (tracks 9)
+    (tracks 11)
     (zones 0)
     (modules 35)
@@
       (padsonsilk false)
       (subtractmaskfromsilk false)
-      (outputformat 1)
+      (outputformat 4)
       (mirror false)
-      (drillshape 1)
+      (drillshape 0)
       (scaleselection 1)
       (outputdirectory ""))
@@
   (module Switch:Sw1 (layer B.Cu)
     (at 126.25 100 90)
-    (fp_text reference SW1 (at 0 -4.4 270) (layer B.SilkS)
+    (fp_text reference SW1 (at 0 -2.5 270) (layer B.SilkS)
       (effects (font (size 1 1) (thickness 0.15)) (justify mirror))
     )
@@
   (via (at 144.75 105.2) (size 0.8) (drill 0.4) (layers F.Cu B.Cu) (net 0))
   (via (at 140 95.15) (size 0.8) (drill 0.4) (layers F.Cu B.Cu) (net 0))
+  (segment (start 138.5 87.5) (end 134.75 87.5) (width 0.25) (layer F.Cu) (net 3))
+  (segment (start 130 87.5) (end 134.05 87.5) (width 0.25) (layer F.Cu) (net 4))
 )

Commit message: minor changes
Parts:
- J2: footprint Switch:MPU-9250 -> Switch:MPU-9250-4pin
- U2: value RFM69HW -> RFM69W
- moved D1 22.5 mm to (171.2, 100.3)
- moved D2 22.5 mm to (171.2, 97.0)
- moved D3 22.5 mm to (171.2, 94.0)
- moved R3 22.5 mm to (166.7, 100.3), turned to 0 degrees
- moved R4 22.5 mm to (166.7, 97.0), turned to 0 degrees
- moved R5 22.5 mm to (166.7, 94.0), turned to 0 degrees
- moved C3 15.0 mm to (142.2, 93.7), turned to 270 degrees
- moved C2 5.91 mm to (142.3, 87.2), turned to 270 degrees
- moved U1 5.55 mm to (151.8, 92.0)
- moved Y1 5.03 mm to (138.4, 90.3), turned to 90 degrees
- moved R1 4.79 mm to (147.8, 77.8)
- moved R2 4.73 mm to (146.0, 79.8)
- moved R6 4.41 mm to (147.7, 82.8)
- moved C10 3.41 mm to (137.4, 102.6)
- moved J4 3.29 mm to (130.7, 109.5), turned to 270 degrees
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Routing:
- net Net-(C3-Pad2): track 4.05 -> 0.00 mm
- net Net-(C2-Pad1): track 3.75 -> 0.00 mm
- net Net-(U2-Pad16): vias 0 -> 1
Other:
- board outline added: 56 x 56 mm

Commit message: small changes
Parts:
- J4: footprint Connector:FanPinHeader_1x03_P2.54mm_Vertical -> Switch:Batt_PHS_Hor_Long18mm
- SW1: footprint Switch:Sw1 -> Switch:Sw_ESP2010
- moved J8 24.1 mm to (145.9, 98.1), turned to 0 degrees
- moved SW1 13.3 mm to (130.5, 87.3), turned to 180 degrees
- moved J4 12.2 mm to (129.3, 97.4), turned to 0 degrees
- moved R6 8.46 mm to (156.1, 82.5), turned to 0 degrees
- moved C10 7.73 mm to (140.2, 109.8), turned to 90 degrees
- moved D4 7.13 mm to (135.5, 99.3), turned to 270 degrees
- moved R1 6.29 mm to (152.3, 82.2), turned to 180 degrees
- moved C8 6.10 mm to (135.9, 119.6)
- moved C11 5.98 mm to (155.8, 99.4)
- moved C9 5.83 mm to (139.3, 113.8)
- moved U3 5.76 mm to (135.6, 113.6)
- moved R2 2.74 mm to (146.7, 82.5)
- moved C2 1.81 mm to (143.5, 85.8)
- moved C3 1.81 mm to (143.4, 92.3)
- moved Y1 1.81 mm to (139.6, 89.0)
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Routing:
- net +3V3: vias 0 -> 1
- net (no net): vias 9 -> 8

Commit message: improuvements
Parts:
- moved C5 22.5 mm to (140.4, 76.5), turned to 0 degrees
- moved J1 21.2 mm to (139.6, 78.8), turned to 270 degrees
- moved J7 10.9 mm to (164.7, 79.7), turned to 0 degrees
- moved J4 3.16 mm to (129.0, 94.2)
- moved J5 1.82 mm to (172.8, 107.7)
- moved C4 1.77 mm to (157.7, 76.0), turned to 180 degrees
- moved C3 1.38 mm to (143.0, 91.0), turned to 90 degrees
- moved C2 1.30 mm to (143.0, 87.0), turned to 90 degrees
- moved R2 0.95 mm to (147.7, 82.5)
- moved J6 0.76 mm to (143.2, 123.8)
- moved IC1 0.72 mm to (167.0, 99.5)
- moved J8 0.62 mm to (145.3, 98.2)
- moved Y1 0.50 mm to (139.1, 89.0)
- moved SW1 0.45 mm to (130.1, 87.5)
- moved R6 0.42 mm to (156.4, 82.2)
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Other:
- outline, holes or cut-outs redrawn

Commit message: minor improvements
Parts:
- J7: value Conn_01x05_Male -> Conn_01x06_Male; footprint Connector_PinHeader_2.54mm:PinHeader_1x05_P2.54mm_Vertical -> Connector_PinHeader_2.54mm:PinHeader_1x06_P2.54mm_Vertical
- J8: value Conn_01x02_Male -> Conn_01x03_Male; footprint Connector_PinHeader_2.54mm:PinHeader_1x02_P2.54mm_Vertical -> Connector_PinHeader_2.54mm:PinHeader_1x03_P2.54mm_Vertical
- U3: footprint Package_TO_SOT_SMD:SOT-23-5 -> Package_TO_SOT_SMD:SOT-23-5_HandSoldering
- moved C7 25.2 mm to (142.2, 103.8)
- moved C6 20.5 mm to (164.7, 113.7)
- moved J7 10.5 mm to (170.8, 88.2), turned to 220 degrees
- moved J5 8.73 mm to (175.6, 99.3), turned to 0 degrees
- moved U2 4.43 mm to (151.6, 112.0), turned to 270 degrees
- moved J8 3.91 mm to (141.6, 99.4), turned to 125 degrees
- moved IC1 3.83 mm to (168.6, 96.0)
- moved J3 3.82 mm to (152.3, 112.0), turned to 270 degrees
- moved C1 3.05 mm to (162.2, 100.4)
- moved J4 2.25 mm to (128.9, 92.0)
- moved J6 2.19 mm to (145.2, 124.7)
- moved C10 1.33 mm to (139.8, 108.5), turned to 0 degrees
- moved R2 1.10 mm to (146.6, 82.5)
- moved R1 1.08 mm to (151.7, 81.6)
- moved C11 1.07 mm to (155.6, 98.3)
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Connections:
- J7 pad 1: /SWCLOCK -> /SWDIO
- J7 pad 2: /SWDIO -> +3V3
- J7 pad 3: /SWO -> /RST
- J7 pad 4: /RST -> /SWCLOCK
- J7 pad 5: GND -> /SWO
- U1 pad 27: Net-(U1-Pad27) -> /CS_RAD
- U1 pad 41: /CS_RAD -> Net-(U1-Pad41)
- U1 pad 46: Net-(U1-Pad46) -> /SWDIO
- U1 pad 50: /SWDIO -> Net-(U1-Pad50)
Routing:
- net +3V3: track 0.00 -> 204.4 mm, vias 1 -> 5
- net GND: track 0.00 -> 144.8 mm, vias 0 -> 2
- net /MOSI: track 0.00 -> 58.5 mm, vias 0 -> 2
- net /MISO: track 0.00 -> 50.4 mm, vias 0 -> 2
- net /SCK: track 0.00 -> 47.8 mm, vias 0 -> 2
- net /CS_RAD: track 0.00 -> 47.2 mm, vias 0 -> 2
- net +BATT: track 0.00 -> 38.1 mm
- net /DIO0: track 0.00 -> 36.5 mm
- net /CS_SD: track 0.00 -> 27.7 mm, vias 0 -> 1
- net /RST: track 0.00 -> 23.7 mm
- net /SCL: track 0.00 -> 17.2 mm
- net Net-(R3-Pad1): track 0.00 -> 15.9 mm, vias 0 -> 1
- net /SWO: track 0.00 -> 14.1 mm
- net /SWDIO: track 0.00 -> 13.8 mm
- net Net-(R4-Pad1): track 0.00 -> 12.2 mm, vias 0 -> 1
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- added copper zone on B.Cu, net GND
- added copper zone on F.Cu, net GND
Other:
- outline, holes or cut-outs redrawn

Commit message: ...
Parts:
- added G***: LOGO, Switch:gjna, B.Cu at (154.7, 90.8)
- added G***: LOGO, Switch:pkiiB, B.Cu at (129.2, 103.8)
- added G***: LOGO, Switch:pkii, B.Cu at (129.2, 103.8)
Routing:
- net GND: vias 2 -> 3
Other:
- board text added: "+"
- board text added: "+3V3"
- board text added: "GND"
- board text added: "RST"
- board text added: "RX"
- board text added: "SWCLK"
- board text added: "SWDIO"
- board text added: "SWO"
- board text added: "TX"

Commit message: ...
Parts:
- moved C10 0.50 mm to (139.2, 108.5)
- moved J8 0.19 mm to (141.4, 99.5)
Routing:
- net +3V3: track 204.4 -> 212.0 mm
- net GND: track 144.8 -> 142.1 mm
Changed lines of the file:
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@@
     (thickness 1.6)
     (drawings 17)
-    (tracks 421)
+    (tracks 420)
     (zones 0)
     (modules 38)
@@
     (31 B.Cu signal)
     (32 B.Adhes user)
-    (33 F.Adhes user)
+    (33 F.Adhes user hide)
     (34 B.Paste user)
     (35 F.Paste user)
@@
       (drillshape 0)
       (scaleselection 1)
-      (outputdirectory "Gerb/"))
+      (outputdirectory "PDFs/"))
   )
   (net 0 "")
@@
   )
   (module Connector_PinHeader_2.54mm:PinHeader_1x03_P2.54mm_Vertical (layer F.Cu)
-    (at 141.569354 99.406884 125)
+    (at 141.45 99.55 125)
     (descr "Through hole straight pin header, 1x03, 2.54mm pitch, single row")
     (tags "Through hole pin header THT 1x03 2.54mm single row")
@@
   )
   (module Capacitor_THT:CP_Radial_D5.0mm_P2.00mm (layer F.Cu)
-    (at 139.75 108.55)
+    (at 139.25 108.55)
     (descr "CP, Radial series, Radial, pin pitch=2.00mm, , diameter=5mm, Electrolytic Capacitor")
     (tags "CP Radial series Radial pin pitch 2.00mm  diameter 5mm Electrolytic Capacitor")
-    (fp_text reference C10 (at -0.1 -3.6) (layer F.SilkS)
+    (fp_text reference C10 (at 0.4 -3.5) (layer F.SilkS)
       (effects (font (size 1 1) (thickness 0.15)))
     )
@@
   (segment (start 160.05 76.575) (end 158.875 75.4) (width 0.4064) (layer F.Cu) (net 1))
   (segment (start 155.1 96.275) (end 155.1 97.118528) (width 0.254) (layer F.Cu) (net 1))
-  (segment (start 141.75 115.75) (end 141.75 108.55) (width 0.635) (layer F.Cu) (net 1))
-  (segment (start 137.9 119.6) (end 141.75 115.75) (width 0.635) (layer F.Cu) (net 1))
-  (segment (start 141.75 110.5625) (end 141.75 108.55) (width 0.635) (layer F.Cu) (net 1))
-  (segment (start 139.65 112.6625) (end 141.75 110.5625) (width 0.635) (layer F.Cu) (net 1))
   (segment (start 132.99 109.41) (end 135.05 109.41) (width 0.635) (layer F.Cu) (net 1))
   (segment (start 131.65 110.75) (end 132.99 109.41) (width 0.635) (layer F.Cu) (net 1))
@@
   (segment (start 150.8 114.25) (end 160.995262 114.25) (width 0.4064) (layer B.Cu) (net 1))
   (segment (start 161.495262 114.75) (end 164.05 114.75) (width 0.4064) (layer B.Cu) (net 1))
-  (segment (start 142.25 108.05) (end 141.75 108.55) (width 0.4064) (layer F.Cu) (net 1))
-  (segment (start 142.25 104.7875) (end 142.25 108.05) (width 0.4064) (layer F.Cu) (net 1))
   (segment (start 162.686597 89.413403) (end 162.65 89.45) (width 0.4064) (layer B.Cu) (net 1))
   (segment (start 162.686597 78.421236) (end 162.686597 89.413403) (width 0.4064) (layer B.Cu) (net 1))
@@
   (via (at 162.35 89.65) (size 1.7) (drill 1) (layers F.Cu B.Cu) (net 1))
   (via (at 138.15 101.05) (size 1.7) (drill 1) (layers F.Cu B.Cu) (net 1))
+  (segment (start 141.25 111.0625) (end 141.25 108.55) (width 0.635) (layer F.Cu) (net 1))
+  (segment (start 139.65 112.6625) (end 141.25 111.0625) (width 0.635) (layer F.Cu) (net 1))
+  (segment (start 141.25 116.25) (end 141.25 111.0625) (width 0.635) (layer F.Cu) (net 1))
+  (segment (start 137.9 119.6) (end 141.25 116.25) (width 0.635) (layer F.Cu) (net 1))
+  (segment (start 142.25 107.55) (end 141.25 108.55) (width 0.635) (layer F.Cu) (net 1))
+  (segment (start 142.25 104.7875) (end 142.25 107.55) (width 0.635) (layer F.Cu) (net 1))
   (via (at 159.85 98.95) (size 1.7) (drill 1) (layers F.Cu B.Cu) (net 2))
   (via (at 139.75 103.55) (size 1.7) (drill 1) (layers F.Cu B.Cu) (net 2))
-  (segment (start 136.65 112.65) (end 139.5 109.8) (width 0.635) (layer F.Cu) (net 2))
   (segment (start 139.9 76.4875) (end 139.8625 76.45) (width 0.254) (layer F.Cu) (net 2))
   (segment (start 149.1 95.4) (end 149.1 96.275) (width 0.254) (layer F.Cu) (net 2))
@@
   (segment (start 143.95 82.05) (end 143.95 83.1) (width 0.4064) (layer F.Cu) (net 2))
   (segment (start 142.85 80.95) (end 143.95 82.05) (width 0.4064) (layer F.Cu) (net 2))
-  (segment (start 139.5 109.8) (end 139.5 108.8) (width 0.635) (layer F.Cu) (net 2))
-  (segment (start 139.75 108.55) (end 139.75 103.55) (width 0.4064) (layer F.Cu) (net 2))
   (segment (start 155.6 96.275) (end 156.375 96.275) (width 0.254) (layer F.Cu) (net 2))
   (segment (start 156.375 96.275) (end 158.75 98.65) (width 0.254) (layer F.Cu) (net 2))
@@
   (segment (start 144.4875 102.9125) (end 144.55 102.85) (width 0.4064) (layer F.Cu) (net 2))
   (segment (start 142.25 102.9125) (end 144.4875 102.9125) (width 0.4064) (layer F.Cu) (net 2))
-  (segment (start 142.953201 106.753201) (end 142.953201 114.553201) (width 0.4064) (layer B.Cu) (net 2))
-  (segment (start 139.75 103.55) (end 142.953201 106.753201) (width 0.4064) (layer B.Cu) (net 2))
-  (segment (start 142.953201 114.553201) (end 143.65 115.25) (width 0.4064) (layer B.Cu) (net 2))
-  (segment (start 143.65 115.25) (end 143.65 115.25) (width 0.4064) (layer B.Cu) (net 2))
-  (via (at 143.65 115.25) (size 1.7) (drill 1) (layers F.Cu B.Cu) (net 2))
-  (segment (start 146.703201 112.196799) (end 143.65 115.25) (width 0.4064) (layer F.Cu) (net 2))
   (segment (start 164.995262 112.65) (end 164.542061 112.196799) (width 0.4064) (layer F.Cu) (net 2))
-  (segment (start 164.542061 112.196799) (end 146.703201 112.196799) (width 0.4064) (layer F.Cu) (net 2))
   (segment (start 166.45 112.65) (end 164.995262 112.65) (width 0.4064) (layer F.Cu) (net 2))
   (segment (start 166.45 112.65) (end 166.45 109.45) (width 0.4064) (layer B.Cu) (net 2))
@@
   (segment (start 162.65 102.05) (end 159.75 99.15) (width 0.4064) (layer B.Cu) (net 2))
   (segment (start 162.65 105.65) (end 162.65 102.05) (width 0.4064) (layer B.Cu) (net 2))
+  (via (at 141.55 118.75) (size 1.7) (drill 1) (layers F.Cu B.Cu) (net 2))
+  (segment (start 148.103201 112.196799) (end 141.55 118.75) (width 0.4064) (layer F.Cu) (net 2))
+  (segment (start 164.542061 112.196799) (end 148.103201 112.196799) (width 0.4064) (layer F.Cu) (net 2))
+  (segment (start 142.953201 117.346799) (end 141.55 118.75) (width 0.4064) (layer B.Cu) (net 2))
+  (segment (start 142.953201 106.753201) (end 142.953201 117.346799) (width 0.4064) (layer B.Cu) (net 2))
+  (segment (start 139.75 103.55) (end 142.953201 106.753201) (width 0.4064) (layer B.Cu) (net 2))
+  (segment (start 139.25 110.3) (end 139.25 108.55) (width 0.635) (layer F.Cu) (net 2))
+  (segment (start 136.9 112.65) (end 139.25 110.3) (width 0.635) (layer F.Cu) (net 2))
+  (segment (start 139.25 104.05) (end 139.75 103.55) (width 0.635) (layer F.Cu) (net 2))
+  (segment (start 139.25 108.55) (end 139.25 104.05) (width 0.635) (layer F.Cu) (net 2))
   (segment (start 143 88.2) (end 143 87.9875) (width 0.25) (layer F.Cu) (net 3))
   (segment (start 143.65 88.85) (end 143 88.2) (width 0.25) (layer F.Cu) (net 3))
@@
   (segment (start 166.093133 85.75) (end 167.584639 84.258494) (width 0.254) (layer F.Cu) (net 34))
   (segment (start 157.05 85.75) (end 166.093133 85.75) (width 0.254) (layer F.Cu) (net 34))
-  (segment (start 141.569354 98.204803) (end 141.569354 99.406884) (width 0.254) (layer F.Cu) (net 35))
-  (segment (start 141.569354 98.080646) (end 141.569354 98.204803) (width 0.254) (layer F.Cu) (net 35))
-  (segment (start 145.3 94.35) (end 141.569354 98.080646) (width 0.254) (layer F.Cu) (net 35))
+  (segment (start 141.45 98.2) (end 141.45 99.55) (width 0.254) (layer F.Cu) (net 35))
+  (segment (start 145.3 94.35) (end 141.45 98.2) (width 0.254) (layer F.Cu) (net 35))
   (segment (start 146.175 94.35) (end 145.3 94.35) (width 0.254) (layer F.Cu) (net 35))
-  (segment (start 146.425 97.95) (end 143.65 97.95) (width 0.254) (layer F.Cu) (net 36))
-  (segment (start 148.1 96.275) (end 146.425 97.95) (width 0.254) (layer F.Cu) (net 36))
+  (segment (start 146.281884 98.093116) (end 143.530646 98.093116) (width 0.254) (layer F.Cu) (net 36))
+  (segment (start 148.1 96.275) (end 146.281884 98.093116) (width 0.254) (layer F.Cu) (net 36))
   (segment (start 156.65 91.85) (end 156 92.5) (width 0.25) (layer F.Cu) (net 37))
   (segment (start 157.525 91.85) (end 156.65 91.85) (width 0.25) (layer F.Cu) (net 37))
@@
     )
   )
-  (zone (net 1) (net_name GND) (layer F.Cu) (hatch edge 0.508)
+  (zone (net 0) (net_name "") (layer B.Cu) (hatch edge 0.508)
     (connect_pads (clearance 0.508))
     (min_thickness 0.254)
-    (fill yes (arc_segments 32) (thermal_gap 0.508) (thermal_bridge_width 0.508))
+    (keepout (tracks not_allowed) (vias not_allowed) (copperpour allowed))
+    (fill (arc_segments 32) (thermal_gap 0.508) (thermal_bridge_width 0.508))
     (polygon
       (pts
-        (xy 184.75 100.85) (xy 167.45 65.85) (xy 124.25 72.25) (xy 116.65 106.55) (xy 134.45 130.55)
-        (xy 172.25 131.45)
+        (xy 125.85 96.95) (xy 132.45 96.95) (xy 132.45 111.05) (xy 125.95 111.05)
       )
     )
   )
-  (zone (net 0) (net_name "") (layer B.Cu) (hatch edge 0.508)
+  (zone (net 1) (net_name GND) (layer F.Cu) (hatch edge 0.508)
     (connect_pads (clearance 0.508))
     (min_thickness 0.254)
-    (keepout (tracks not_allowed) (vias not_allowed) (copperpour allowed))
-    (fill (arc_segments 32) (thermal_gap 0.508) (thermal_bridge_width 0.508))
+    (fill yes (arc_segments 32) (thermal_gap 0.508) (thermal_bridge_width 0.508))
     (polygon
       (pts
-        (xy 125.85 96.95) (xy 132.45 96.95) (xy 132.45 111.05) (xy 125.95 111.05)
+        (xy 180.65 82.35) (xy 179.85 108.45) (xy 170.85 131.95) (xy 133.35 129.95) (xy 115.95 104.45)
+        (xy 126.75 75.65) (xy 155.15 66.15) (xy 180.55 82.55)
       )
     )
@@
     (polygon
       (pts
-        (xy 149.75 66.25) (xy 182.95 84.45) (xy 177.65 126.35) (xy 137.15 131.55) (xy 115.95 104.05)
-        (xy 127.95 73.35)
+        (xy 183.35 111.65) (xy 163.65 132.45) (xy 118.35 124.75) (xy 115.15 89.05) (xy 138.45 66.25)
+        (xy 171.75 72.75) (xy 182.85 96.15) (xy 183.45 111.95) (xy 183.25 111.75)
       )
     )
