File: Probe/Hardware/CanSat2020ProbeS/CanSat2020Probe.sch (KiCad schematic (older format))
At the start: 33 parts, among them IC1 TESEO-LIV3F, J1 BME280, J2 MPU-9250, J3 Micro_SD_Card, J4 Conn_01x03_Male, J5 Conn_Coaxial, J6 Conn_Coaxial, J7 Conn_01x05_Male, J8 Conn_01x03_Male, U1 STM32F411RETx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

Commit message: new parts and reorganisation
Parts:
- C10, C8: footprint Capacitor_SMD:CP_Elec_8x10 -> Capacitor_THT:CP_Radial_D5.0mm_P2.00mm
Changed lines of the file:
@@
 F 0 "C8" H 3215 6746 50  0000 L CNN
 F 1 "47uF" H 3215 6655 50  0000 L CNN
-F 2 "Capacitor_SMD:CP_Elec_8x10" H 3138 6550 50  0001 C CNN
+F 2 "Capacitor_THT:CP_Radial_D5.0mm_P2.00mm" H 3138 6550 50  0001 C CNN
 F 3 "~" H 3100 6700 50  0001 C CNN
 	1    3100 6700
@@
 F 0 "C10" H 4565 6746 50  0000 L CNN
 F 1 "47uF" H 4565 6655 50  0000 L CNN
-F 2 "Capacitor_SMD:CP_Elec_8x10" H 4488 6550 50  0001 C CNN
+F 2 "Capacitor_THT:CP_Radial_D5.0mm_P2.00mm" H 4488 6550 50  0001 C CNN
 F 3 "~" H 4450 6700 50  0001 C CNN
 	1    4450 6700

Commit message: upadte
Parts:
- added C11: 4.7uF, Capacitor_SMD:C_0805_2012Metric, symbol Device:C
- added SW1: SW_DIP_x01, Switch:Sw1, symbol Switch:SW_DIP_x01
- J1: footprint Connector_PinHeader_2.54mm:PinHeader_1x04_P2.54mm_Vertical -> Switch:BME280
- J2: footprint Connector_PinHeader_2.54mm:PinHeader_1x10_P2.54mm_Vertical -> Switch:MPU-9250
- J5, J6: footprint Connector_Coaxial:U.FL_Molex_MCRF_73412-0110_Vertical -> Connector_Coaxial:U.FL_Hirose_U.FL-R-SMT-1_Vertical
- J8: value Conn_01x03_Male -> Conn_01x02_Male; footprint Connector_PinHeader_2.54mm:PinHeader_1x03_P2.54mm_Vertical -> Connector_PinHeader_2.54mm:PinHeader_1x02_P2.54mm_Vertical; symbol Connector:Conn_01x03_Male -> Connector:Conn_01x02_Male
Connections:
- net +BATT: now also SW1.1; no longer J4.1 (Pin_1)
- net DBGRX: now also J8.2 (Pin_2); no longer J8.3 (Pin_3)
- net DBGTX: now also J8.1 (Pin_1); no longer J8.2 (Pin_2)
- net GND: now also C11.2; no longer J8.1 (Pin_1)
- net at U1.30 (VCAP1): now also C11.1
- new net: J4.1 (Pin_1), SW1.2
- no-connect marks 55 -> 54
Other:
- moved on the sheet: C10, C6, C8, C9, D4, J3, J4, J7, U3

Commit message: Impprovements
Other:
- moved on the sheet: C1, C4, C5, C6, C7, IC1, J5, J6, U2

Commit message: minor changes
Parts:
- removed U2: RFM69HW, RF_Module:HOPERF_RFM69HW, symbol RF_Module:RFM69HW
- added U2: RFM69W, RF_Module:HOPERF_RFM69HW, symbol RF_Module:RFM69W
- J2: footprint Switch:MPU-9250 -> Switch:MPU-9250-4pin
Connections:
- net +3V3: now also U2.8 (3.3V)
- net CS_RAD: now also U2.15 (NSS)
- net DIO0: now also U2.2 (DIO0)
- net GND: now also U2.11 (GND), U2.9 (GND)
- net MISO: now also U2.13 (MISO)
- net MOSI: now also U2.14 (MOSI)
- net SCK: now also U2.12 (SCK)
- net at J6.1 (In): now also U2.10 (ANA)
Changed lines of the file:
@@
 F 0 "J2" H 6350 5500 50  0000 L CNN
 F 1 "MPU-9250" H 6350 5400 50  0000 L CNN
-F 2 "Switch:MPU-9250" H 6500 4850 50  0001 C CNN
+F 2 "Switch:MPU-9250-4pin" H 6500 4850 50  0001 C CNN
 F 3 "~" H 6500 4850 50  0001 C CNN
 	1    6500 4850
@@
 Wire Wire Line
 	9150 900  9150 950
-Wire Wire Line
-	9250 2050 9250 2200
-$Comp
-L power:GND #PWR0115
-U 1 1 5DE007C8
-P 9250 2200
-F 0 "#PWR0115" H 9250 1950 50  0001 C CNN
-F 1 "GND" H 9255 2027 50  0000 C CNN
-F 2 "" H 9250 2200 50  0001 C CNN
-F 3 "" H 9250 2200 50  0001 C CNN
-	1    9250 2200
-	1    0    0    -1
-$EndComp
 $Comp
 L Connector:Conn_Coaxial J5
@@
 Wire Wire Line
 	8650 1450 8250 1450
-Text Label 8250 1450 0    50   ~ 0
-MOSI
-Text Label 8250 1350 0    50   ~ 0
-MISO
 Wire Wire Line
 	8650 1250 8250 1250
@@
 Text Label 8250 1550 0    50   ~ 0
 CS_RAD
-Wire Wire Line
-	9650 1350 9900 1350
-Text Label 9900 1350 0    50   ~ 0
-DIO0
 Wire Wire Line
 	5450 1300 5200 1300
@@
 NoConn ~ 9650 1850
 NoConn ~ 9650 1750
-$Comp
-L RF_Module:RFM69HW U2
-U 1 1 5DC7018C
-P 9150 1550
-F 0 "U2" H 8800 2150 50  0000 C CNN
-F 1 "RFM69HW" H 8800 2050 50  0000 C CNN
-F 2 "RF_Module:HOPERF_RFM69HW" H 9150 950 50  0001 C CNN
-F 3 "https://www.hoperf.com/data/upload/portal/20181127/5bfcbb56f1fd7.pdf" H 9150 1250 50  0001 C CNN
-	1    9150 1550
-	1    0    0    -1
-$EndComp
 NoConn ~ 9650 1650
 NoConn ~ 9650 1550
@@
 	1    0    0    -1
 $EndComp
+Text Label 9900 1350 0    50   ~ 0
+DIO0
+Wire Wire Line
+	9650 1350 9900 1350
+Text Label 8250 1450 0    50   ~ 0
+MOSI
+Text Label 8250 1350 0    50   ~ 0
+MISO
+$Comp
+L power:GND #PWR0115
+U 1 1 5DE007C8
+P 9250 2200
+F 0 "#PWR0115" H 9250 1950 50  0001 C CNN
+F 1 "GND" H 9255 2027 50  0000 C CNN
+F 2 "" H 9250 2200 50  0001 C CNN
+F 3 "" H 9250 2200 50  0001 C CNN
+	1    9250 2200
+	1    0    0    -1
+$EndComp
+Wire Wire Line
+	9250 2050 9250 2200
+$Comp
+L RF_Module:RFM69W U2
+U 1 1 5E226D7C
+P 9150 1550
+F 0 "U2" H 8850 2200 50  0000 C CNN
+F 1 "RFM69W" H 8850 2100 50  0000 C CNN
+F 2 "RF_Module:HOPERF_RFM69HW" H 9150 950 50  0001 C CNN
+F 3 "https://www.hoperf.com/data/upload/portal/20181127/5bfcbe34756e1.pdf" H 9150 1250 50  0001 C CNN
+	1    9150 1550
+	1    0    0    -1
+$EndComp

Commit message: small changes
Parts:
- J4: footprint Connector:FanPinHeader_1x03_P2.54mm_Vertical -> Switch:Batt_PHS_Hor_Long18mm
- SW1: footprint Switch:Sw1 -> Switch:Sw_ESP2010
Changed lines of the file:
@@
 F 0 "J4" H 1458 6931 50  0000 C CNN
 F 1 "Conn_01x03_Male" H 1450 6850 50  0000 C CNN
-F 2 "Connector:FanPinHeader_1x03_P2.54mm_Vertical" H 1350 6650 50  0001 C CNN
+F 2 "Switch:Batt_PHS_Hor_Long18mm" H 1350 6650 50  0001 C CNN
 F 3 "~" H 1350 6650 50  0001 C CNN
 	1    1350 6650
@@
 F 0 "SW1" H 2250 6300 50  0000 C CNN
 F 1 "SW_DIP_x01" H 2250 6400 50  0000 C CNN
-F 2 "Switch:Sw1" H 2250 6550 50  0001 C CNN
+F 2 "Switch:Sw_ESP2010" H 2250 6550 50  0001 C CNN
 F 3 "~" H 2250 6550 50  0001 C CNN
 	1    2250 6550

Commit message: minor improvements
Parts:
- removed J7: Conn_01x05_Male, Connector_PinHeader_2.54mm:PinHeader_1x05_P2.54mm_Vertical, symbol Connector:Conn_01x05_Male
- removed J8: Conn_01x02_Male, Connector_PinHeader_2.54mm:PinHeader_1x02_P2.54mm_Vertical, symbol Connector:Conn_01x02_Male
- added J7: Conn_01x06_Male, Connector_PinHeader_2.54mm:PinHeader_1x06_P2.54mm_Vertical, symbol Connector:Conn_01x06_Male
- added J8: Conn_01x03_Male, Connector_PinHeader_2.54mm:PinHeader_1x03_P2.54mm_Vertical, symbol Connector:Conn_01x03_Male
- U3: footprint Package_TO_SOT_SMD:SOT-23-5 -> Package_TO_SOT_SMD:SOT-23-5_HandSoldering
Connections:
- net +3V3: now also J7.2 (Pin_2)
- net CS_RAD: now also U1.27 (PB1); no longer U1.41 (PA8)
- net DBGRX: now also J8.2 (Pin_2)
- net DBGTX: now also J8.1 (Pin_1)
- net GND: now also J7.6 (Pin_6), J8.3 (Pin_3)
- net RST: now also J7.3 (Pin_3)
- net SWCLOCK: now also J7.4 (Pin_4)
- net SWDIO: now also U1.46 (PA13), J7.1 (Pin_1); no longer U1.50 (PA15)
- net SWO: now also J7.5 (Pin_5)
Changed lines of the file:
@@
 encoding utf-8
 Sheet 1 1
-Title "Píseň kosmická 2"
+Title "Píseň kosmická II"
 Date "2020-12-28"
-Rev "v01"
+Rev "v02"
 Comp ""
 Comment1 ""
@@
 F 0 "U3" H 3750 6992 50  0000 C CNN
 F 1 "LD3985M33R_SOT23" H 3750 6901 50  0000 C CNN
-F 2 "Package_TO_SOT_SMD:SOT-23-5" H 3750 6975 50  0001 C CIN
+F 2 "Package_TO_SOT_SMD:SOT-23-5_HandSoldering" H 3750 6975 50  0001 C CIN
 F 3 "http://www.st.com/internet/com/TECHNICAL_RESOURCES/TECHNICAL_LITERATURE/DATASHEET/CD00003395.pdf" H 3750 6650 50  0001 C CNN
 	1    3750 6650
@@
 CS_SD
 $Comp
-L Connector:Conn_01x02_Male J8
-U 1 1 5DE8C9E8
-P 2400 1150
-F 0 "J8" H 2450 1400 50  0000 R CNN
-F 1 "Conn_01x02_Male" H 2750 1300 50  0000 R CNN
-F 2 "Connector_PinHeader_2.54mm:PinHeader_1x02_P2.54mm_Vertical" H 2400 1150 50  0001 C CNN
-F 3 "~" H 2400 1150 50  0001 C CNN
-	1    2400 1150
-	1    0    0    -1
-$EndComp
-$Comp
 L Device:C C5
 U 1 1 5E052D24
@@
 Wire Wire Line
 	2800 7100 2800 7150
-Wire Wire Line
-	1200 1100 1450 1100
-Text Label 1450 1100 0    50   ~ 0
+Text Label 1450 1300 0    50   ~ 0
 SWCLOCK
-Text Label 1450 1200 0    50   ~ 0
+Text Label 1450 1000 0    50   ~ 0
 SWDIO
-Text Label 1450 1300 0    50   ~ 0
+Text Label 1450 1400 0    50   ~ 0
 SWO
 Wire Wire Line
@@
 	1050 3250 1050 3200
 Wire Wire Line
-	1200 1500 1500 1500
-Wire Wire Line
-	1500 1500 1500 1550
+	1200 1500 1450 1500
+Wire Wire Line
+	1450 1500 1450 1550
 $Comp
 L power:GND #PWR0137
@@
 NoConn ~ 4100 2150
 NoConn ~ 4100 3250
-NoConn ~ 4100 3350
 NoConn ~ 4100 3750
-NoConn ~ 4100 3850
 NoConn ~ 4100 3950
 NoConn ~ 4100 4150
@@
 NoConn ~ 4100 4450
 NoConn ~ 4100 4750
-NoConn ~ 4100 4850
 NoConn ~ 4100 4950
 NoConn ~ 4100 5050
@@
 Text Label 4150 4050 0    50   ~ 0
 SWO
-Text Label 4500 3550 0    50   ~ 0
+Text Label 4500 3350 0    50   ~ 0
 SWDIO
 Text Label 4500 3450 0    50   ~ 0
 SWCLOCK
-Wire Wire Line
-	4100 2850 4500 2850
 Wire Wire Line
 	1200 1400 1450 1400
@@
 Text Label 2200 2050 0    50   ~ 0
 RST
-Text Label 1450 1400 0    50   ~ 0
+Text Label 1450 1200 0    50   ~ 0
 RST
 $Comp
 L power:GND #PWR0132
 U 1 1 5E1C680C
-P 1500 1550
-F 0 "#PWR0132" H 1500 1300 50  0001 C CNN
-F 1 "GND" V 1505 1422 50  0000 R CNN
-F 2 "" H 1500 1550 50  0001 C CNN
-F 3 "" H 1500 1550 50  0001 C CNN
-	1    1500 1550
+P 1450 1550
+F 0 "#PWR0132" H 1450 1300 50  0001 C CNN
+F 1 "GND" V 1455 1422 50  0000 R CNN
+F 2 "" H 1450 1550 50  0001 C CNN
+F 3 "" H 1450 1550 50  0001 C CNN
+	1    1450 1550
 	1    0    0    -1
 $EndComp
@@
 	4100 3050 4500 3050
 Wire Wire Line
-	4100 3550 4500 3550
-Wire Wire Line
 	4100 3450 4500 3450
 Wire Wire Line
@@
 Wire Wire Line
 	2700 2050 2200 2050
-$Comp
-L Connector:Conn_01x05_Male J7
-U 1 1 5DE8D72E
-P 1000 1300
-F 0 "J7" H 1108 1681 50  0000 C CNN
-F 1 "Conn_01x05_Male" H 1108 1590 50  0000 C CNN
-F 2 "Connector_PinHeader_2.54mm:PinHeader_1x05_P2.54mm_Vertical" H 1000 1300 50  0001 C CNN
-F 3 "~" H 1000 1300 50  0001 C CNN
-	1    1000 1300
-	1    0    0    -1
-$EndComp
 Wire Wire Line
 	4100 2450 4500 2450
@@
 Text Label 4500 2950 0    50   ~ 0
 RX
-Text Label 4500 2850 0    50   ~ 0
+Text Label 4500 3850 0    50   ~ 0
 CS_RAD
 Text Label 4500 3050 0    50   ~ 0
@@
 P 4350 4000
 F 0 "#PWR0118" H 4350 3850 50  0001 C CNN
-F 1 "+3V3" H 4365 4173 50  0000 C CNN
+F 1 "+3V3" H 4450 3950 50  0000 C CNN
 F 2 "" H 4350 4000 50  0001 C CNN
 F 3 "" H 4350 4000 50  0001 C CNN
@@
 P 4650 4050
 F 0 "#PWR0117" H 4650 3900 50  0001 C CNN
-F 1 "+3V3" H 4665 4223 50  0000 C CNN
+F 1 "+3V3" H 4750 4000 50  0000 C CNN
 F 2 "" H 4650 4050 50  0001 C CNN
 F 3 "" H 4650 4050 50  0001 C CNN
@@
 	1    0    0    -1
 $EndComp
+NoConn ~ 4100 3550
+Wire Wire Line
+	4500 3350 4100 3350
+$Comp
+L Connector:Conn_01x06_Male J7
+U 1 1 5E4112AB
+P 1000 1200
+F 0 "J7" H 1050 1650 50  0000 C CNN
+F 1 "Conn_01x06_Male" H 1050 1550 50  0000 C CNN
+F 2 "Connector_PinHeader_2.54mm:PinHeader_1x06_P2.54mm_Vertical" H 1000 1200 50  0001 C CNN
+F 3 "~" H 1000 1200 50  0001 C CNN
+	1    1000 1200
+	1    0    0    -1
+$EndComp
+$Comp
+L power:+3V3 #PWR0134
+U 1 1 5E4290A9
+P 1800 1000
+F 0 "#PWR0134" H 1800 850 50  0001 C CNN
+F 1 "+3V3" H 1815 1173 50  0000 C CNN
+F 2 "" H 1800 1000 50  0001 C CNN
+F 3 "" H 1800 1000 50  0001 C CNN
+	1    1800 1000
+	1    0    0    -1
+$EndComp
+$Comp
+L Connector:Conn_01x03_Male J8
+U 1 1 5E32C6CF
+P 2400 1250
+F 0 "J8" H 2500 1600 50  0000 C CNN
+F 1 "Conn_01x03_Male" H 2500 1500 50  0000 C CNN
+F 2 "Connector_PinHeader_2.54mm:PinHeader_1x03_P2.54mm_Vertical" H 2400 1250 50  0001 C CNN
+F 3 "~" H 2400 1250 50  0001 C CNN
+	1    2400 1250
+	1    0    0    -1
+$EndComp
+$Comp
+L power:GND #PWR0138
+U 1 1 5E3377AE
+P 2800 1400
+F 0 "#PWR0138" H 2800 1150 50  0001 C CNN
+F 1 "GND" H 2805 1227 50  0000 C CNN
+F 2 "" H 2800 1400 50  0001 C CNN
+F 3 "" H 2800 1400 50  0001 C CNN
+	1    2800 1400
+	1    0    0    -1
+$EndComp
+Wire Wire Line
+	2600 1350 2800 1350
+Wire Wire Line
+	2800 1350 2800 1400
+NoConn ~ 4100 4850
+Wire Wire Line
+	4100 3850 4500 3850
+NoConn ~ 4100 2850
+Wire Wire Line
+	1200 1000 1450 1000
+Wire Wire Line
+	1800 1100 1800 1000
+Wire Wire Line
+	1200 1100 1800 1100
 $EndSCHEMATC

Commit message: ...
Other:
- note added: "Connectors"
- note added: "GPS"
- note added: "Gyroscope, accelerometer and magnetometer module"
- note added: "MCU"
- note added: "Power suply"
- note added: "Radio"
- note added: "SD card"
- note added: "Temperature, humidity and pressure modele"
- moved on the sheet: C1, C10, C11, C2, C3, C4, C5, C6, C7, C8, C9, D1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
